Commit message: Update URDF file

File: src/my_robot_description/urdf/simple-joint.urdf (robot description, URDF)
Before this commit: robot Simple_Arm, 2 links, 1 joints
Links:
- added link left_arm; visual box size=0.1 0.1 0.4
- added link right_arm; visual box size=0.1 0.1 0.4
Joints:
- removed joint base_to_arm
- added joint base_to_head: type revolute, parent base, child head, origin xyz=0 0 0.25, axis 0 0 1, limit lower=-1.5708 upper=1.5708 effort=30 velocity=1.0
- added joint base_to_left_arm: type revolute, parent base, child left_arm, origin xyz=-0.25 0 -0.05, axis 1 0 0, limit lower=-1.5708 upper=1.5708 effort=30 velocity=1.0
- added joint base_to_right_arm: type revolute, parent base, child right_arm, origin xyz=0.25 0 -0.05, axis 1 0 0, limit lower=-1.5708 upper=1.5708 effort=30 velocity=1.0
