Commit message: Added Optimus Bot

File: src/gazebo_tutorial/urdf/teslabot.urdf.xacro (robot description, xacro)
@@ -1,129 +1,254 @@
 <?xml version="1.0"?>
-<robot xmlns:xacro="http://www.ros.org/wiki/xacro" name="teslabot">
-  <xacro:property name="base_length" value="0.6"/>
-  <xacro:property name="base_width" value="0.4"/>
-  <xacro:property name="base_height" value="0.2"/>
-  <xacro:property name="wheel_radius" value="0.1"/>
-  <xacro:property name="wheel_width" value="0.05"/>
-  <material name="blue">
-    <color rgba="0.2 0.2 0.8 1.0"/>
-  </material>
-  <material name="black">
-    <color rgba="0.1 0.1 0.1 1.0"/>
-  </material>
-  <link name="base_link">
-    <visual>
-      <geometry>
-        <box size="${base_length} ${base_width} ${base_height}"/>
-      </geometry>
-      <material name="blue"/>
-    </visual>
-    <collision>
-      <geometry>
-        <box size="${base_length} ${base_width} ${base_height}"/>
-      </geometry>
-    </collision>
-    <inertial>
-      <mass value="5.0"/>
-      <inertia ixx="0.1" ixy="0.0" ixz="0.0" iyy="0.1" iyz="0.0" izz="0.1"/>
-    </inertial>
-  </link>
-  <xacro:macro name="wheel" params="prefix y_offset">
-    <link name="${prefix}_wheel">
-      <visual>
-        <origin rpy="${pi/2} 0 0" xyz="0 0 0"/>
-        <geometry>
-          <cylinder radius="${wheel_radius}" length="${wheel_width}"/>
-        </geometry>
-        <material name="black"/>
-      </visual>
-      <collision>
-        <origin rpy="${pi/2} 0 0" xyz="0 0 0"/>
-        <geometry>
-          <cylinder radius="${wheel_radius}" length="${wheel_width}"/>
-        </geometry>
-      </collision>
-      <inertial>
-        <mass value="0.5"/>
-        <inertia ixx="0.001" ixy="0.0" ixz="0.0" iyy="0.001" iyz="0.0" izz="0.001"/>
-      </inertial>
-    </link>
-    <joint name="${prefix}_wheel_joint" type="continuous">
-      <parent link="base_link"/>
-      <child link="${prefix}_wheel"/>
-      <origin xyz="0 ${y_offset} ${-base_height/2}" rpy="0 0 0"/>
-      <axis xyz="0 1 0"/>
-    </joint>
-  </xacro:macro>
-  <xacro:wheel prefix="left" y_offset="${base_width/2 + wheel_width/2}"/>
-  <xacro:wheel prefix="right" y_offset="${-(base_width/2 + wheel_width/2)}"/>
-  <!-- Caster supports keep the 2-wheeled base from tipping over -->
-  <xacro:macro name="caster" params="prefix x_offset">
-    <link name="${prefix}_caster">
-      <visual>
-        <geometry>
-          <sphere radius="${wheel_radius}"/>
-        </geometry>
-        <material name="black"/>
-      </visual>
-      <collision>
-        <geometry>
-          <sphere radius="${wheel_radius}"/>
-        </geometry>
-      </collision>
-      <inertial>
-        <mass value="0.2"/>
-        <inertia ixx="0.0001" ixy="0.0" ixz="0.0" iyy="0.0001" iyz="0.0" izz="0.0001"/>
-      </inertial>
-    </link>
-    <joint name="${prefix}_caster_joint" type="fixed">
-      <parent link="base_link"/>
-      <child link="${prefix}_caster"/>
-      <origin xyz="${x_offset} 0 ${-base_height/2}" rpy="0 0 0"/>
-    </joint>
-  </xacro:macro>
-  <xacro:caster prefix="front" x_offset="${base_length/2 - wheel_radius}"/>
-  <xacro:caster prefix="back" x_offset="${-(base_length/2 - wheel_radius)}"/>
-  <!-- Gazebo: high friction on drive wheels, near-zero on casters so they slide -->
-  <gazebo reference="left_wheel">
-    <mu1>1.0</mu1>
-    <mu2>1.0</mu2>
+<robot name="robot" xmlns:xacro="http://ros.org/wiki/xacro">
+  <link name="world"/>
+  <link name="head">
+    <inertial>
+      <mass value="1"/>
+      <inertia ixx=".1" ixy="0" ixz="0" iyy=".1" iyz="0" izz=".1" />
+    </inertial>
+    <visual>
+      <origin xyz="0 0 0" rpy="0 0 0" />
+      <geometry>
+        <!-- <cylinder radius="0.01" length=".5" /> -->
+        <mesh filename="$(find gazebo_tutorial)/meshes/head.STL" scale="1 1 1"/>
+      </geometry>
+      <material name="black">
+        <color rgba="0 0 0 1"/> <!-- Black color -->
+      </material>
+    </visual>
+  </link>
+  <joint name="world_to_head" type="fixed">
+    <origin xyz="0 0 1" />
+    <parent link="world"/>
+    <child link="head"/>
+  </joint>
+  <link name="body">
+    <inertial>
+      <mass value="1"/>
+      <inertia ixx=".1" ixy="0" ixz="0" iyy=".1" iyz="0" izz=".1" />
+    </inertial>
+    <visual>
+      <origin xyz="0 0 0" rpy="0 0 0" />
+      <geometry>
+        <mesh filename="$(find gazebo_tutorial)/meshes/body.STL" scale="1 1 1"/>
+      </geometry>
+      <material name="gray">
+        <color rgba=".2 .2 .2 1" />
+      </material>
+    </visual>
+  </link>
+  <joint name="head_to_body" type="fixed">
+    <origin xyz="0 0 0" />
+    <parent link="head"/>
+    <child link="body"/>
+  </joint>
+  <link name="shoulder_right">
+    <inertial>
+      <mass value="1"/>
+      <inertia ixx=".1" ixy="0" ixz="0" iyy=".1" iyz="0" izz=".1" />
+    </inertial>
+    <visual>
+      <origin xyz="0 0 0" rpy="0 0 0" />
+      <geometry>
+        <mesh filename="$(find gazebo_tutorial)/meshes/shoulder.STL" scale="1 1 1"/>
+      </geometry>
+      <material name="gray">
+        <color rgba=".2 .2 .2 1" />
+      </material>
+    </visual>
+  </link>
+  <joint name="body_to_shoulder_right" type="revolute">
+    <origin xyz="0.206 0 -0.0635" rpy="-${pi/2} 0 0"/>
+    <parent link="body"/>
+    <child link="shoulder_right"/>
+    <axis rpy="0 0 0" xyz="0 0 1"/>
+    <limit lower="-${pi}" upper="${pi}" effort="100" velocity="20"/>
+  </joint>
+  <link name="shoulder_left">
+    <inertial>
+      <mass value="1"/>
+      <inertia ixx=".1" ixy="0" ixz="0" iyy=".1" iyz="0" izz=".1" />
+    </inertial>
+    <visual>
+      <origin xyz="0 0 0" rpy="0 0 0" />
+      <geometry>
+        <mesh filename="$(find gazebo_tutorial)/meshes/shoulder.STL" scale="1 1 1"/>
+      </geometry>
+      <material name="gray">
+        <color rgba=".2 .2 .2 1" />
+      </material>
+    </visual>
+  </link>
+  <joint name="body_to_shoulder_left" type="revolute">
+    <origin xyz="-0.206 0 -0.0635" rpy="${pi/2} 0 ${pi}"/>
+    <parent link="body"/>
+    <child link="shoulder_left"/>
+    <axis rpy="0 0 0" xyz="0 0 1"/>
+    <limit lower="-${pi}" upper="${pi}" effort="100" velocity="20"/>
+  </joint>
+  <link name="arm_upper_right">
+    <inertial>
+      <mass value="1"/>
+      <inertia ixx=".1" ixy="0" ixz="0" iyy=".1" iyz="0" izz=".1" />
+    </inertial>
+    <visual>
+      <origin xyz="0 0 0" rpy="0 0 0" />
+      <geometry>
+        <mesh filename="$(find gazebo_tutorial)/meshes/arm_upper.STL" scale="1 1 1"/>
+      </geometry>
+      <material name="gray">
+        <color rgba=".2 .2 .2 1" />
+      </material>
+    </visual>
+  </link>
+  <joint name="shoulder_to_arm_upper_right" type="revolute">
+    <origin xyz="0 0 0" rpy="0 0 ${pi}"/>
+    <parent link="shoulder_right"/>
+    <child link="arm_upper_right"/>
+    <axis rpy="0 0 0" xyz="0 0 1"/>
+    <limit lower="-${pi}" upper="${pi}" effort="100" velocity="20"/>
+  </joint>
+  <link name="arm_upper_left">
+    <inertial>
+      <mass value="1"/>
+      <inertia ixx=".1" ixy="0" ixz="0" iyy=".1" iyz="0" izz=".1" />
+    </inertial>
+    <visual>
+      <origin xyz="0 0 0" rpy="0 0 0" />
+      <geometry>
+        <mesh filename="$(find gazebo_tutorial)/meshes/arm_upper.STL" scale="1 1 1"/>
+      </geometry>
+      <material name="gray">
+        <color rgba=".2 .2 .2 1" />
+      </material>
+    </visual>
+  </link>
+  <joint name="shoulder_to_arm_upper_left" type="revolute">
+    <origin xyz="0 0 0" rpy="0 0 0"/>
+    <parent link="shoulder_left"/>
+    <child link="arm_upper_left"/>
+    <axis rpy="0 0 0" xyz="0 0 1"/>
+    <limit lower="-${pi}" upper="${pi}" effort="100" velocity="20"/>
+  </joint>
+  <link name="arm_lower_right">
+    <inertial>
+      <mass value="1"/>
+      <inertia ixx=".1" ixy="0" ixz="0" iyy=".1" iyz="0" izz=".1" />
+    </inertial>
+    <visual>
+      <origin xyz="0 0 0" rpy="0 0 0" />
+      <geometry>
+        <mesh filename="$(find gazebo_tutorial)/meshes/arm_lower.STL" scale="1 1 1"/>
+      </geometry>
+      <material name="gray">
+        <color rgba=".2 .2 .2 1" />
+      </material>
+    </visual>
+  </link>
+  <joint name="arm_upper_to_lower_right" type="revolute">
+    <origin xyz="0 -.358 0" rpy="0 -${pi/2} 0"/>
+    <parent link="arm_upper_right"/>
+    <child link="arm_lower_right"/>
+    <axis rpy="0 0 0" xyz="0 0 1"/>
+    <limit lower="-${pi}" upper="${pi}" effort="100" velocity="20"/>
+  </joint>
+  <link name="arm_lower_left">
+    <inertial>
+      <mass value="1"/>
+      <inertia ixx=".1" ixy="0" ixz="0" iyy=".1" iyz="0" izz=".1" />
+    </inertial>
+    <visual>
+      <origin xyz="0 0 0" rpy="0 0 0" />
+      <geometry>
+        <mesh filename="$(find gazebo_tutorial)/meshes/arm_lower.STL" scale="1 1 1"/>
+      </geometry>
+      <material name="gray">
+        <color rgba=".2 .2 .2 1" />
+      </material>
+    </visual>
+  </link>
+  <joint name="arm_upper_to_lower_left" type="revolute">
+    <origin xyz="0 -.358 0" rpy="0 ${pi/2} 0"/>
+    <parent link="arm_upper_left"/>
+    <child link="arm_lower_left"/>
+    <axis rpy="0 0 0" xyz="0 0 1"/>
+    <limit lower="-${pi}" upper="${pi}" effort="100" velocity="20"/>
+  </joint>
+  <link name="hand_right">
+    <inertial>
+      <mass value="1"/>
+      <inertia ixx=".1" ixy="0" ixz="0" iyy=".1" iyz="0" izz=".1" />
+    </inertial>
+    <visual>
+      <origin xyz="0 0 0" rpy="0 0 0" />
+      <geometry>
+        <mesh filename="$(find gazebo_tutorial)/meshes/hand_right.STL" scale="1 1 1"/>
+      </geometry>
+      <material name="gray">
+        <color rgba=".2 .2 .2 1" />
+      </material>
+    </visual>
+  </link>
+  <joint name="arm_lower_to_hand_right" type="fixed">
+    <origin xyz="0 -.338 0" rpy="${pi/2} -${pi} 0"/>
+    <parent link="arm_lower_right"/>
+    <child link="hand_right"/>
+  </joint>
+  <link name="hand_left">
+    <inertial>
+      <mass value="1"/>
+      <inertia ixx=".1" ixy="0" ixz="0" iyy=".1" iyz="0" izz=".1" />
+    </inertial>
+    <visual>
+      <origin xyz="0 0 0" rpy="0 0 0" />
+      <geometry>
+        <mesh filename="$(find gazebo_tutorial)/meshes/hand_left.STL" scale="1 1 1"/>
+      </geometry>
+      <material name="gray">
+        <color rgba=".2 .2 .2 1" />
+      </material>
+    </visual>
+  </link>
+  <joint name="arm_lower_to_hand_left" type="fixed">
+    <origin xyz="0 -.338 0" rpy="${pi/2} 0 0"/>
+    <parent link="arm_lower_left"/>
+    <child link="hand_left"/>
+  </joint>
+  <gazebo reference="head">
     <material>Gazebo/Black</material>
   </gazebo>
-  <gazebo reference="right_wheel">
-    <mu1>1.0</mu1>
-    <mu2>1.0</mu2>
-    <material>Gazebo/Black</material>
+  <gazebo reference="body">
+    <material>Gazebo/White</material>
   </gazebo>
-  <gazebo reference="front_caster">
-    <mu1>0.0</mu1>
-    <mu2>0.0</mu2>
-    <material>Gazebo/Black</material>
-  </gazebo>
-  <gazebo reference="back_caster">
-    <mu1>0.0</mu1>
-    <mu2>0.0</mu2>
-    <material>Gazebo/Black</material>
-  </gazebo>
-  <gazebo reference="base_link">
-    <material>Gazebo/Blue</material>
-  </gazebo>
-  <!-- Differential drive: subscribes to /cmd_vel, drives the wheels, publishes odom -->
+  <ros2_control name="GazeboSystem" type="system">
+    <hardware>
+      <plugin>gazebo_ros2_control/GazeboSystem</plugin>
+    </hardware>
+    <joint name="arm_upper_to_lower_right">
+      <command_interface name="position">
+        <param name="min">-3.14</param>
+        <param name="max">3.14</param>
+      </command_interface>
+      <state_interface name="position">
+        <param name="initial_value">0</param>
+      </state_interface>
+      <state_interface name="velocity"/>
+      <state_interface name="effort"/>
+    </joint>
+    <joint name="arm_upper_to_lower_left">
+      <command_interface name="position">
+        <param name="min">-3.14</param>
+        <param name="max">3.14</param>
+      </command_interface>
+      <state_interface name="position">
+        <param name="initial_value">0</param>
+      </state_interface>
+      <state_interface name="velocity"/>
+      <state_interface name="effort"/>
+    </joint>
+  </ros2_control>
   <gazebo>
-    <plugin name="diff_drive" filename="libgazebo_ros_diff_drive.so">
-      <update_rate>30</update_rate>
-      <left_joint>left_wheel_joint</left_joint>
-      <right_joint>right_wheel_joint</right_joint>
-      <wheel_separation>${base_width + wheel_width}</wheel_separation>
-      <wheel_diameter>${2 * wheel_radius}</wheel_diameter>
-      <max_wheel_torque>20</max_wheel_torque>
-      <max_wheel_acceleration>1.0</max_wheel_acceleration>
-      <command_topic>cmd_vel</command_topic>
-      <publish_odom>true</publish_odom>
-      <publish_odom_tf>true</publish_odom_tf>
-      <publish_wheel_tf>true</publish_wheel_tf>
-      <odometry_topic>odom</odometry_topic>
-      <odometry_frame>odom</odometry_frame>
-      <robot_base_frame>base_link</robot_base_frame>
+    <plugin filename="libgazebo_ros2_control.so" name="gazebo_ros2_control">
+      <parameters>$(find gazebo_tutorial)/config/joint_controller.yaml</parameters>
     </plugin>
   </gazebo>

Commit message: update Optimus movement

File: src/gazebo_tutorial/urdf/teslabot.urdf.xacro (robot description, xacro)
@@ -11,5 +11,5 @@
       <geometry>
         <!-- <cylinder radius="0.01" length=".5" /> -->
-        <mesh filename="$(find gazebo_tutorial)/meshes/head.STL" scale="1 1 1"/>
+        <mesh filename="$(find gazebo_tutorial)/meshes/Optimus/head.STL" scale="1 1 1"/>
       </geometry>
       <material name="black">
@@ -31,5 +31,5 @@
       <origin xyz="0 0 0" rpy="0 0 0" />
       <geometry>
-        <mesh filename="$(find gazebo_tutorial)/meshes/body.STL" scale="1 1 1"/>
+        <mesh filename="$(find gazebo_tutorial)/meshes/Optimus/torso.STL" scale="1 1 1"/>
       </geometry>
       <material name="gray">
@@ -51,5 +51,5 @@
       <origin xyz="0 0 0" rpy="0 0 0" />
       <geometry>
-        <mesh filename="$(find gazebo_tutorial)/meshes/shoulder.STL" scale="1 1 1"/>
+        <mesh filename="$(find gazebo_tutorial)/meshes/Optimus/shoulder.STL" scale="1 1 1"/>
       </geometry>
       <material name="gray">
@@ -73,5 +73,5 @@
       <origin xyz="0 0 0" rpy="0 0 0" />
       <geometry>
-        <mesh filename="$(find gazebo_tutorial)/meshes/shoulder.STL" scale="1 1 1"/>
+        <mesh filename="$(find gazebo_tutorial)/meshes/Optimus/shoulder.STL" scale="1 1 1"/>
       </geometry>
       <material name="gray">
@@ -95,5 +95,5 @@
       <origin xyz="0 0 0" rpy="0 0 0" />
       <geometry>
-        <mesh filename="$(find gazebo_tutorial)/meshes/arm_upper.STL" scale="1 1 1"/>
+        <mesh filename="$(find gazebo_tutorial)/meshes/Optimus/arm_upper.STL" scale="1 1 1"/>
       </geometry>
       <material name="gray">
@@ -117,5 +117,5 @@
       <origin xyz="0 0 0" rpy="0 0 0" />
       <geometry>
-        <mesh filename="$(find gazebo_tutorial)/meshes/arm_upper.STL" scale="1 1 1"/>
+        <mesh filename="$(find gazebo_tutorial)/meshes/Optimus/arm_upper.STL" scale="1 1 1"/>
       </geometry>
       <material name="gray">
@@ -139,5 +139,5 @@
       <origin xyz="0 0 0" rpy="0 0 0" />
       <geometry>
-        <mesh filename="$(find gazebo_tutorial)/meshes/arm_lower.STL" scale="1 1 1"/>
+        <mesh filename="$(find gazebo_tutorial)/meshes/Optimus/arm_lower.STL" scale="1 1 1"/>
       </geometry>
       <material name="gray">
@@ -161,5 +161,5 @@
       <origin xyz="0 0 0" rpy="0 0 0" />
       <geometry>
-        <mesh filename="$(find gazebo_tutorial)/meshes/arm_lower.STL" scale="1 1 1"/>
+        <mesh filename="$(find gazebo_tutorial)/meshes/Optimus/arm_lower.STL" scale="1 1 1"/>
       </geometry>
       <material name="gray">
@@ -183,5 +183,5 @@
       <origin xyz="0 0 0" rpy="0 0 0" />
       <geometry>
-        <mesh filename="$(find gazebo_tutorial)/meshes/hand_right.STL" scale="1 1 1"/>
+        <mesh filename="$(find gazebo_tutorial)/meshes/Optimus/hand_right.STL" scale="1 1 1"/>
       </geometry>
       <material name="gray">
@@ -203,5 +203,5 @@
       <origin xyz="0 0 0" rpy="0 0 0" />
       <geometry>
-        <mesh filename="$(find gazebo_tutorial)/meshes/hand_left.STL" scale="1 1 1"/>
+        <mesh filename="$(find gazebo_tutorial)/meshes/Optimus/hand_left.STL" scale="1 1 1"/>
       </geometry>
       <material name="gray">

Commit message: Update

File: src/gazebo_tutorial/urdf/teslabot.urdf.xacro (robot description, xacro)
@@ -11,5 +11,5 @@
       <geometry>
         <!-- <cylinder radius="0.01" length=".5" /> -->
-        <mesh filename="$(find gazebo_tutorial)/meshes/Optimus/head.STL" scale="1 1 1"/>
+        <mesh filename="file://$(find gazebo_tutorial)/meshes/Optimus/head.STL" scale="1 1 1"/>
       </geometry>
       <material name="black">
@@ -19,5 +19,5 @@
   </link>
   <joint name="world_to_head" type="fixed">
-    <origin xyz="0 0 1" />
+    <origin xyz="0 0 1.5" />
     <parent link="world"/>
     <child link="head"/>
@@ -31,5 +31,5 @@
       <origin xyz="0 0 0" rpy="0 0 0" />
       <geometry>
-        <mesh filename="$(find gazebo_tutorial)/meshes/Optimus/torso.STL" scale="1 1 1"/>
+        <mesh filename="file://$(find gazebo_tutorial)/meshes/Optimus/torso.STL" scale="1 1 1"/>
       </geometry>
       <material name="gray">
@@ -51,5 +51,5 @@
       <origin xyz="0 0 0" rpy="0 0 0" />
       <geometry>
-        <mesh filename="$(find gazebo_tutorial)/meshes/Optimus/shoulder.STL" scale="1 1 1"/>
+        <mesh filename="file://$(find gazebo_tutorial)/meshes/Optimus/shoulder.STL" scale="1 1 1"/>
       </geometry>
       <material name="gray">
@@ -73,5 +73,5 @@
       <origin xyz="0 0 0" rpy="0 0 0" />
       <geometry>
-        <mesh filename="$(find gazebo_tutorial)/meshes/Optimus/shoulder.STL" scale="1 1 1"/>
+        <mesh filename="file://$(find gazebo_tutorial)/meshes/Optimus/shoulder.STL" scale="1 1 1"/>
       </geometry>
       <material name="gray">
@@ -95,5 +95,5 @@
       <origin xyz="0 0 0" rpy="0 0 0" />
       <geometry>
-        <mesh filename="$(find gazebo_tutorial)/meshes/Optimus/arm_upper.STL" scale="1 1 1"/>
+        <mesh filename="file://$(find gazebo_tutorial)/meshes/Optimus/arm_upper.STL" scale="1 1 1"/>
       </geometry>
       <material name="gray">
@@ -117,5 +117,5 @@
       <origin xyz="0 0 0" rpy="0 0 0" />
       <geometry>
-        <mesh filename="$(find gazebo_tutorial)/meshes/Optimus/arm_upper.STL" scale="1 1 1"/>
+        <mesh filename="file://$(find gazebo_tutorial)/meshes/Optimus/arm_upper.STL" scale="1 1 1"/>
       </geometry>
       <material name="gray">
@@ -139,5 +139,5 @@
       <origin xyz="0 0 0" rpy="0 0 0" />
       <geometry>
-        <mesh filename="$(find gazebo_tutorial)/meshes/Optimus/arm_lower.STL" scale="1 1 1"/>
+        <mesh filename="file://$(find gazebo_tutorial)/meshes/Optimus/arm_lower.STL" scale="1 1 1"/>
       </geometry>
       <material name="gray">
@@ -161,5 +161,5 @@
       <origin xyz="0 0 0" rpy="0 0 0" />
       <geometry>
-        <mesh filename="$(find gazebo_tutorial)/meshes/Optimus/arm_lower.STL" scale="1 1 1"/>
+        <mesh filename="file://$(find gazebo_tutorial)/meshes/Optimus/arm_lower.STL" scale="1 1 1"/>
       </geometry>
       <material name="gray">
@@ -183,5 +183,5 @@
       <origin xyz="0 0 0" rpy="0 0 0" />
       <geometry>
-        <mesh filename="$(find gazebo_tutorial)/meshes/Optimus/hand_right.STL" scale="1 1 1"/>
+        <mesh filename="file://$(find gazebo_tutorial)/meshes/Optimus/hand_right.STL" scale="1 1 1"/>
       </geometry>
       <material name="gray">
@@ -203,5 +203,5 @@
       <origin xyz="0 0 0" rpy="0 0 0" />
       <geometry>
-        <mesh filename="$(find gazebo_tutorial)/meshes/Optimus/hand_left.STL" scale="1 1 1"/>
+        <mesh filename="file://$(find gazebo_tutorial)/meshes/Optimus/hand_left.STL" scale="1 1 1"/>
       </geometry>
       <material name="gray">
@@ -248,25 +248,25 @@
     </joint>
   </ros2_control>
-  <gazebo reference = "head">
-    <sensor type = "camera" name = "camera">
-        <pose>0 0 0.25 0 0.7 1.5707</pose>
-        <visualize>true</visualize>
-        <update_rate>5</update_rate>
-        <camera>
-            <horizontal_fov>1</horizontal_fov>
-            <image>
-                <format>R8G8B8</format>
-                <width>640</width>
-                <height>480</height>
-            </image>
-            <clip>
-                <near>0.05</near>
-                <far>1.0</far>
-            </clip>
-        </camera>
-        <plugin filename="libgazebo_ros2_camera.so" name="gazebo_ros2_camera">
-            <frame_name>world_to_head</frame_name>
-        </plugin>
-    </sensor>
+  <gazebo reference="head">
+      <sensor name="camera" type="camera">
+          <pose> 0 0 0.25 0 0.7 1.5707</pose>
+          <visualize>true</visualize>
+          <update_rate>5</update_rate>
+          <camera>
+              <horizontal_fov>1</horizontal_fov>
+              <image>
+                  <format>R8G8B8</format>
+                  <width>640</width>
+                  <height>480</height>
+              </image>
+              <clip>
+                  <near>0.05</near>
+                  <far>1</far>
+              </clip>
+          </camera>
+          <plugin name="camera_controller" filename="libgazebo_ros_camera.so">
+              <frame_name>world_to_head</frame_name>
+          </plugin>
+      </sensor>
   </gazebo>
   <gazebo>
